File: IOX_Monitor.kicad_pcb (KiCad board)
At the start: 2 copper layers, 33 x 48.3 mm, 30 parts, among them J1 Conn_01x02, J2 Conn_01x08, J3 Conn_01x08, J4 Conn_01x08, J5 Conn_01x08, J6 Conn_01x08, Q1 DMG2301L, Q2 DMG2301L, Q3 DMG2301L, Q4 DMG2301L, Q5 DMG2301L, Q6 DMG2301L, Q7 DMG2301L, Q8 DMG2301L

Commit message: P-FET & Sockets
Parts:
- J4, J5, J6: footprint Connector_PinHeader_2.54mm:PinHeader_1x08_P2.54mm_Vertical -> Connector_PinSocket_2.54mm:PinSocket_1x08_P2.54mm_Vertical
- Q1, Q2, Q3, Q4, Q5, Q6, Q7, Q8: value DMG2301L -> Q_P-FET_2.3A_SOT-23_2301V
