File: IOX_Monitor.kicad_sch (KiCad schematic)
At the start: 30 parts, among them J1 Conn_01x02, J2 Conn_01x08, J3 Conn_01x08, J4 Conn_01x08, J5 Conn_01x08, J6 Conn_01x08, Q1 DMG2301L, Q2 DMG2301L, Q3 DMG2301L, Q4 DMG2301L, Q5 DMG2301L, Q6 DMG2301L, Q7 DMG2301L, Q8 DMG2301L

Commit message: P-FET & Sockets
Parts:
- J4, J5, J6: footprint Connector_PinHeader_2.54mm:PinHeader_1x08_P2.54mm_Vertical -> (none); symbol SPCoast:Conn_01x08 -> SPCoast:Conn_01x08_Socket
- Q1, Q2, Q3, Q4, Q5, Q6, Q7, Q8: value DMG2301L -> Q_P-FET_2.3A_SOT-23_2301V
Other:
- company: MRCS -> SPCoast
- title: cpNode IOX Testbed -> IOX Monitor
Changed lines of the file:
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@@
 	(paper "USLetter")
 	(title_block
-		(title "cpNode IOX Testbed")
+		(title "IOX Monitor")
 		(date "2026.07")
 		(rev "1.0")
-		(company "MRCS")
+		(company "SPCoast")
 		(comment 1 "John Plocher")
-		(comment 2 "IOX Plugin")
+		(comment 2 "IOX LED Monitor and test point breakout")
+		(comment 9 "active")
 	)
 	(text "GND"
@@
 			)
 		)
-		(property "Value" "DMG2301L"
+		(property "Value" "Q_P-FET_2.3A_SOT-23_2301V"
 			(at 123.19 90.1699 0)
+			(hide yes)
 			(show_name no)
 			(do_not_autoplace no)
@@
 	)
 	(symbol
-		(lib_id "SPCoast:Conn_01x08")
+		(lib_id "SPCoast:Conn_01x08_Socket")
 		(at 224.79 67.31 270)
 		(mirror x)
@@
 			)
 		)
-		(property "Footprint" "Connector_PinHeader_2.54mm:PinHeader_1x08_P2.54mm_Vertical"
+		(property "Footprint" ""
 			(at 224.79 67.31 0)
 			(hide yes)
@@
 		)
 		(property "Datasheet" ""
-			(at 225.044 68.834 0)
+			(at 224.79 67.31 0)
 			(hide yes)
 			(show_name no)
@@
 		)
 		(property "Description" "Generic connector, single row, 01x08, script generated"
-			(at 237.49 69.342 0)
+			(at 224.79 67.31 0)
 			(hide yes)
 			(show_name no)
@@
 		(in_pos_files yes)
 		(dnp no)
-		(fields_autoplaced yes)
 		(property "Reference" "Q1"
 			(at 199.39 86.3599 0)
@@
 			)
 		)
-		(property "Value" "DMG2301L"
-			(at 199.39 88.8999 0)
+		(property "Value" "Q_P-FET_2.3A_SOT-23_2301V"
+			(at 218.694 93.218 0)
 			(show_name no)
 			(do_not_autoplace no)
@@
 		(in_pos_files yes)
 		(dnp no)
-		(fields_autoplaced yes)
 		(property "Reference" "#P+014"
 			(at 127 82.55 0)
@@
 		)
 		(property "Value" "+5V"
-			(at 124.46 87.63 90)
+			(at 124.46 86.614 90)
 			(show_name no)
 			(do_not_autoplace no)
@@
 			)
 		)
-		(property "Value" "DMG2301L"
+		(property "Value" "Q_P-FET_2.3A_SOT-23_2301V"
 			(at 142.24 88.8999 0)
+			(hide yes)
 			(show_name no)
 			(do_not_autoplace no)
@@
 		(in_pos_files yes)
 		(dnp no)
-		(fields_autoplaced yes)
 		(property "Reference" "#P+013"
 			(at 146.05 82.55 0)
@@
 		)
 		(property "Value" "+5V"
-			(at 143.51 87.63 90)
+			(at 143.51 85.852 90)
 			(show_name no)
 			(do_not_autoplace no)
@@
 	)
 	(symbol
-		(lib_id "SPCoast:Conn_01x08")
+		(lib_id "SPCoast:Conn_01x08_Socket")
 		(at 144.78 67.31 270)
 		(mirror x)
@@
 			)
 		)
-		(property "Footprint" "Connector_PinHeader_2.54mm:PinHeader_1x08_P2.54mm_Vertical"
+		(property "Footprint" ""
 			(at 144.78 67.31 0)
 			(hide yes)
@@
 		)
 		(property "Datasheet" ""
-			(at 145.034 68.834 0)
+			(at 144.78 67.31 0)
 			(hide yes)
 			(show_name no)
@@
 		)
 		(property "Description" "Generic connector, single row, 01x08, script generated"
-			(at 157.48 69.342 0)
+			(at 144.78 67.31 0)
 			(hide yes)
 			(show_name no)
@@
 			)
 		)
-		(property "Value" "DMG2301L"
+		(property "Value" "Q_P-FET_2.3A_SOT-23_2301V"
 			(at 180.34 88.8999 0)
+			(hide yes)
 			(show_name no)
 			(do_not_autoplace no)
@@
 			)
 		)
-		(property "Value" "DMG2301L"
+		(property "Value" "Q_P-FET_2.3A_SOT-23_2301V"
 			(at 104.14 88.8999 0)
+			(hide yes)
 			(show_name no)
 			(do_not_autoplace no)
@@
 			)
 		)
-		(property "Value" "DMG2301L"
+		(property "Value" "Q_P-FET_2.3A_SOT-23_2301V"
 			(at 161.29 88.8999 0)
+			(hide yes)
 			(show_name no)
 			(do_not_autoplace no)
@@
 		(in_pos_files yes)
 		(dnp no)
-		(fields_autoplaced yes)
 		(property "Reference" "#P+011"
 			(at 184.15 82.55 0)
@@
 		)
 		(property "Value" "+5V"
-			(at 181.61 87.63 90)
+			(at 181.61 85.852 90)
 			(show_name no)
 			(do_not_autoplace no)
@@
 			)
 		)
-		(property "Value" "DMG2301L"
+		(property "Value" "Q_P-FET_2.3A_SOT-23_2301V"
 			(at 66.04 88.8999 0)
+			(hide yes)
 			(show_name no)
 			(do_not_autoplace no)
@@
 			)
 		)
-		(property "Value" "DMG2301L"
+		(property "Value" "Q_P-FET_2.3A_SOT-23_2301V"
 			(at 85.09 88.8999 0)
+			(hide yes)
 			(show_name no)
 			(do_not_autoplace no)
@@
 	)
 	(symbol
-		(lib_id "SPCoast:Conn_01x08")
+		(lib_id "SPCoast:Conn_01x08_Socket")
 		(at 187.96 67.31 270)
 		(mirror x)
@@
 			)
 		)
-		(property "Footprint" "Connector_PinHeader_2.54mm:PinHeader_1x08_P2.54mm_Vertical"
+		(property "Footprint" ""
 			(at 187.96 67.31 0)
 			(hide yes)
@@
 		)
 		(property "Datasheet" ""
-			(at 188.214 68.834 0)
+			(at 187.96 67.31 0)
 			(hide yes)
 			(show_name no)
@@
 		)
 		(property "Description" "Generic connector, single row, 01x08, script generated"
-			(at 200.66 69.342 0)
+			(at 187.96 67.31 0)
 			(hide yes)
 			(show_name no)
@@
 		(in_pos_files yes)
 		(dnp no)
-		(fields_autoplaced yes)
 		(property "Reference" "#P+012"
 			(at 165.1 82.55 0)
@@
 		)
 		(property "Value" "+5V"
-			(at 162.56 87.63 90)
+			(at 162.56 85.852 90)
 			(show_name no)
 			(do_not_autoplace no)
@@
 		(in_pos_files yes)
 		(dnp no)
-		(fields_autoplaced yes)
 		(property "Reference" "#P+010"
 			(at 203.2 82.55 0)
@@
 		)
 		(property "Value" "+5V"
-			(at 200.66 87.63 90)
+			(at 200.66 85.852 90)
 			(show_name no)
 			(do_not_autoplace no)
